File: PCB/microUPDI_isolated.kicad_pcb (KiCad board)
At the start: 2 copper layers, 40.2 x 41.1 mm, 34 parts, among them J1 SUPPLY_VOLTAGE_SWITCH, J2 UPDI_ISO, J3 UPDI, J4 ISP, Q1 BC817, Q2 BC817, Q3 BC817, U1 AMS1117-3.3, U2 B0505S-1W, U3 ADuM1250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

Commit message: Update readme and PCB
Parts:
- added C8: 10u, Capacitor_Tantalum_SMD:CP_EIA-3528-21_Kemet-B, B.Cu at (140.2, 75.1)
- added C9: 10u, Capacitor_Tantalum_SMD:CP_EIA-3528-21_Kemet-B, B.Cu at (146.1, 74.2)
- moved R2 3.82 mm to (149.6, 77.2), turned to 180 degrees
Routing:
- net Net-(U2-VIN): track 28.0 -> 30.8 mm
- net +5V_ISO: track 25.8 -> 27.5 mm
