File: PCB/microUPDI_isolated.kicad_sch (KiCad schematic)
At the start: 34 parts, among them J1 SUPPLY_VOLTAGE_SWITCH, J2 UPDI_ISO, J3 UPDI, J4 ISP, Q1 BC817, Q2 BC817, Q3 BC817, U1 AMS1117-3.3, U2 B0505S-1W, U3 ADuM1250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

Commit message: Update readme and PCB
Parts:
- added C8, C9: 10u, Capacitor_Tantalum_SMD:CP_EIA-3528-21_Kemet-B, symbol Device:C
Connections:
- net +5V_ISO: now also C9.1
- net GND: now also C8.2, C9.2
- net at F1.1, R3.1, R4.1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: now also C8.1
